File: 4k-keypad/4k-keypad.kicad_sch (KiCad schematic)
At the start: 24 parts, among them SW1 SW_Push, U1 ATmega32U4-A, Y1 16MHz

Commit message: update commit
Parts:
- F1: value Polyfuse_Small -> 500mA
- SW1: value SW_Push -> Reset
Connections:
- net COL0: now also U1.29 (PB5)
- net COL1: now also U1.28 (PB4)
- net ROW0: now also U1.30 (PB6)
- net ROW1: now also U1.27 (PD7)
- no-connect marks 1 -> 2
Changed lines of the file:
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@@
   )
   (no_connect (at 66.675 58.42))
+  (no_connect (at 147.955 49.53))
   (wire (pts (xy 147.955 41.91) (xy 154.94 41.91))
     (stroke (width 0) (type default) (color 0 0 0 0))
@@
     )
   )
+  (global_label "COL1" (shape input) (at 97.155 53.34 0) (fields_autoplaced)
+    (effects (font (size 1.27 1.27)) (justify left))
+    (property "Intersheet References" "${INTERSHEET_REFS}" (id 0) (at 104.4062 53.2606 0)
+      (effects (font (size 1.27 1.27)) (justify left) hide)
+    )
+  )
   (global_label "ROW0" (shape input) (at 143.51 92.71 180) (fields_autoplaced)
     (effects (font (size 1.27 1.27)) (justify right))
@@
     )
   )
+  (global_label "ROW1" (shape input) (at 97.155 91.44 0) (fields_autoplaced)
+    (effects (font (size 1.27 1.27)) (justify left))
+    (property "Intersheet References" "${INTERSHEET_REFS}" (id 0) (at 104.8295 91.3606 0)
+      (effects (font (size 1.27 1.27)) (justify left) hide)
+    )
+  )
+  (global_label "COL0" (shape input) (at 97.155 55.88 0) (fields_autoplaced)
+    (effects (font (size 1.27 1.27)) (justify left))
+    (property "Intersheet References" "${INTERSHEET_REFS}" (id 0) (at 104.4062 55.8006 0)
+      (effects (font (size 1.27 1.27)) (justify left) hide)
+    )
+  )
   (global_label "D+" (shape input) (at 154.94 46.99 0) (fields_autoplaced)
     (effects (font (size 1.27 1.27)) (justify left))
@@
     )
   )
+  (global_label "ROW0" (shape input) (at 97.155 58.42 0) (fields_autoplaced)
+    (effects (font (size 1.27 1.27)) (justify left))
+    (property "Intersheet References" "${INTERSHEET_REFS}" (id 0) (at 104.8295 58.3406 0)
+      (effects (font (size 1.27 1.27)) (justify left) hide)
+    )
+  )
   (global_label "ROW1" (shape input) (at 143.51 110.49 180) (fields_autoplaced)
     (effects (font (size 1.27 1.27)) (justify right))
@@
   )
   (symbol (lib_id "Device:C_Small") (at 47.625 46.99 90) (unit 1)
-    (in_bom yes) (on_board yes) (fields_autoplaced)
-    (property "Reference" "C1" (id 0) (at 47.6313 40.64 90))
-    (property "Value" "22pF" (id 1) (at 47.6313 43.18 90))
+    (in_bom yes) (on_board yes)
+    (property "Reference" "C1" (id 0) (at 47.625 45.72 90))
+    (property "Value" "22pF" (id 1) (at 47.625 48.26 90))
     (property "Footprint" "Capacitor_SMD:C_0805_2012Metric" (id 2) (at 47.625 46.99 0)
       (effects (font (size 1.27 1.27)) hide)
@@
     (in_bom yes) (on_board yes) (fields_autoplaced)
     (property "Reference" "F1" (id 0) (at 164.465 35.56 90))
-    (property "Value" "Polyfuse_Small" (id 1) (at 164.465 38.1 90))
+    (property "Value" "500mA" (id 1) (at 164.465 38.1 90))
     (property "Footprint" "Fuse:Fuse_1206_3216Metric" (id 2) (at 169.545 40.64 0)
       (effects (font (size 1.27 1.27)) (justify left) hide)
@@
   )
   (symbol (lib_id "Device:C_Small") (at 47.625 53.975 90) (unit 1)
-    (in_bom yes) (on_board yes) (fields_autoplaced)
-    (property "Reference" "C2" (id 0) (at 47.6313 46.99 90))
-    (property "Value" "22pF" (id 1) (at 47.6313 49.53 90))
+    (in_bom yes) (on_board yes)
+    (property "Reference" "C2" (id 0) (at 47.625 52.705 90))
+    (property "Value" "22pF" (id 1) (at 47.625 55.245 90))
     (property "Footprint" "Capacitor_SMD:C_0805_2012Metric" (id 2) (at 47.625 53.975 0)
       (effects (font (size 1.27 1.27)) hide)
@@
   )
   (symbol (lib_id "power:+5V") (at 54.61 63.5 0) (unit 1)
-    (in_bom yes) (on_board yes) (fields_autoplaced)
+    (in_bom yes) (on_board yes)
     (property "Reference" "#PWR0107" (id 0) (at 54.61 67.31 0)
       (effects (font (size 1.27 1.27)) hide)
     )
-    (property "Value" "+5V" (id 1) (at 54.61 57.785 0))
+    (property "Value" "+5V" (id 1) (at 54.61 60.325 0))
     (property "Footprint" "" (id 2) (at 54.61 63.5 0)
       (effects (font (size 1.27 1.27)) hide)
@@
   (symbol (lib_id "Switch:SW_Push") (at 34.29 43.18 0) (unit 1)
     (in_bom yes) (on_board yes) (fields_autoplaced)
-    (property "Reference" "SW1" (id 0) (at 34.29 34.925 0))
-    (property "Value" "SW_Push" (id 1) (at 34.29 37.465 0))
+    (property "Reference" "SW1" (id 0) (at 34.29 35.56 0))
+    (property "Value" "Reset" (id 1) (at 34.29 38.1 0))
     (property "Footprint" "random-keyboard-parts:SKQG-1155865" (id 2) (at 34.29 38.1 0)
       (effects (font (size 1.27 1.27)) hide)
@@
     )
     (path "/959e8eaf-825f-4b69-afcb-d255cedf52a2"
-      (reference "F1") (unit 1) (value "Polyfuse_Small") (footprint "Fuse:Fuse_1206_3216Metric")
+      (reference "F1") (unit 1) (value "500mA") (footprint "Fuse:Fuse_1206_3216Metric")
     )
     (path "/2796166b-08b0-4dd8-a300-c2fb2273d50e"
@@
     )
     (path "/f4a2cfc0-3daa-4926-ac70-5caf4f976ed6"
-      (reference "SW1") (unit 1) (value "SW_Push") (footprint "random-keyboard-parts:SKQG-1155865")
+      (reference "SW1") (unit 1) (value "Reset") (footprint "random-keyboard-parts:SKQG-1155865")
     )
     (path "/f83663bf-f8f8-45ed-8057-ced26e1c8768"
